File: hardware/DMXLEDs.kicad_sch (KiCad schematic)
At the start: 16 parts

Commit message: Update
Parts:
- renumbered D405 to D402, D409 to D403, D413 to D404, D402 to D405, D410 to D407, D414 to D408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
