File: hardware/DMXOut.kicad_sch (KiCad schematic)
At the start: 3 parts, among them J201 SJ2-25404B-SMT-TR, U201 THVD2442

Commit message: Replace diode
Other:
- title: DMX Out -> V2 dmx

Commit message: Update
Parts:
- C201: Id (none) -> Capacitor:${SYMBOL_NAME}
- J201: Id (none) -> Audio:${SYMBOL_NAME}; Rating (none) -> 2.5mm
- U201: Id (none) -> RS485:${SYMBOL_NAME}; Rating (none) -> 20Mbps
Changed lines of the file:
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@@
 	(title_block
 		(title "V2 dmx")
-		(date "2026-03-30")
+		(date "2026-04-14")
 		(rev "2026-03-30")
 		(company "Versio Duo")
+		(comment 1 "MIDI to DMX Bridge")
 	)
 	(rectangle
@@
 			)
 		)
+		(property "Id" "RS485:${SYMBOL_NAME}"
+			(at 128.27 142.24 0)
+			(hide yes)
+			(show_name no)
+			(do_not_autoplace no)
+			(effects
+				(font
+					(size 1.27 1.27)
+				)
+			)
+		)
+		(property "Rating" "20Mbps"
+			(at 129.54 149.86 0)
+			(hide yes)
+			(show_name no)
+			(do_not_autoplace no)
+			(effects
+				(font
+					(size 1.27 1.27)
+				)
+			)
+		)
 		(pin "1"
 		)
@@
 			)
 		)
+		(property "Id" "Audio:${SYMBOL_NAME}"
+			(at 172.72 90.17 0)
+			(hide yes)
+			(show_name no)
+			(do_not_autoplace no)
+			(effects
+				(font
+					(size 1.27 1.27)
+				)
+			)
+		)
+		(property "Rating" "2.5mm"
+			(at 172.72 77.47 0)
+			(hide yes)
+			(show_name no)
+			(do_not_autoplace no)
+			(effects
+				(font
+					(size 1.27 1.27)
+				)
+			)
+		)
 		(pin "1"
 		)
@@
 			(hide yes)
 			(show_name no)
+			(do_not_autoplace no)
+			(effects
+				(font
+					(size 1.27 1.27)
+				)
+			)
+		)
+		(property "Id" "Capacitor:${SYMBOL_NAME}"
+			(at 148.59 105.41 0)
+			(hide yes)
+			(show_name no)

Commit message: Good Bye Imperial
Parts:
- C201: footprint V2_Capacitor_SMD:C_0603 -> V2_Capacitor_SMD:C_1608; symbol V2_Capacitor:0603_0u1 -> V2_Capacitor:1608_0u1
Changed lines of the file:
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@@
 	(title_block
 		(title "V2 dmx")
-		(date "2026-04-14")
+		(date "2026-05-11")
 		(rev "2026-03-30")
 		(company "Versio Duo")
@@
 	)
 	(symbol
-		(lib_id "V2_Capacitor:0603_0u1")
+		(lib_id "V2_Capacitor:1608_0u1")
 		(at 148.59 90.17 0)
 		(unit 1)
@@
 			)
 		)
-		(property "Footprint" "V2_Capacitor_SMD:C_0603"
+		(property "Footprint" "V2_Capacitor_SMD:C_1608"
 			(at 148.59 107.188 0)
 			(hide yes)
