File: hardware/DMXOut.kicad_sch (KiCad schematic)
At the start: 3 parts, among them J201 SJ2-25404B-SMT-TR, U201 THVD2442

Commit message: Refresh
Changed lines of the file:
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@@
 	(title_block
 		(title "V2 dmx")
-		(date "2026-05-19")
+		(date "2026-05-27")
 		(rev "2026-03-30")
 		(company "Versio Duo")
@@
 		)
 		(property "Value" "+3V3"
-			(at 125.476 82.804 0)
-			(show_name no)
-			(do_not_autoplace no)
-			(effects
-				(font
-					(size 1.27 1.27)
-				)
-				(justify left)
+			(at 128.27 82.296 0)
+			(show_name no)
+			(do_not_autoplace no)
+			(effects
+				(font
+					(size 1.27 1.27)
+					(color 255 92 187 1)
+				)
 			)
 		)
@@
 				(font
 					(size 1.27 1.27)
+					(color 255 92 187 1)
 				)
 			)
@@
 				(font
 					(size 1.27 1.27)
-				)
-			)
+					(color 255 92 187 1)
+				)
+			)
