File: hardware/MIDIIn.kicad_sch (KiCad schematic)
At the start: 6 parts, among them J301 SJ2-25404B-SMT-TR, U301 TLP2361

Commit message: Replace diode
Parts:
- D301: value RB501SM -> PMEG2010EPK; footprint V2_Diode_SMD:D_SOD-523 -> V2_Diode_SMD:D_SOD-1608; symbol V2_Diode:RB501SM -> V2_Diode:PMEG2010EPK; Manufacturer ROHM Semiconductor -> Nexperia; Mouser 755-RB501SM-30FHT2R -> 771-PMEG2010EPK; Product RB501SM-30FHT2R -> PMEG2010EPK; Rating (none) -> 20V
Other:
- title: MIDI In -> V2 dmx
Changed lines of the file:
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@@
 (kicad_sch
-	(version 20250114)
+	(version 20260306)
 	(generator "eeschema")
-	(generator_version "9.0")
+	(generator_version "10.0")
 	(paper "A4")
 	(title_block
-		(title "MIDI In")
-		(date "2025-09-19")
-		(rev "3")
+		(title "V2 dmx")
+		(date "2026-03-30")
+		(rev "2026-03-30")
 	)

Commit message: Update
Parts:
- C301, C302: Id (none) -> Capacitor:${SYMBOL_NAME}
- D301: Id (none) -> Diode:${SYMBOL_NAME}
- J301: Id (none) -> Audio:${SYMBOL_NAME}; Rating (none) -> 2.5mm
- R301: Id (none) -> Resistor:${SYMBOL_NAME}
- U301: Id (none) -> Optocoupler:${SYMBOL_NAME}; Rating (none) -> 15Mbps
Other:
- company: (none) -> Versio Duo
Changed lines of the file:
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@@
 	(title_block
 		(title "V2 dmx")
-		(date "2026-03-30")
+		(date "2026-04-14")
 		(rev "2026-03-30")
+		(company "Versio Duo")
+		(comment 1 "MIDI to DMX Bridge")
 	)

Commit message: Update
Parts:
- renumbered C302 to C301, C301 to C302

Commit message: Good Bye Imperial
Parts:
- C301, C302: footprint V2_Capacitor_SMD:C_0603 -> V2_Capacitor_SMD:C_1608; symbol V2_Capacitor:0603_0u1 -> V2_Capacitor:1608_0u1
- R301: footprint V2_Resistor_SMD:R_0603 -> V2_Resistor_SMD:R_1608; symbol V2_Resistor:0603_220R -> V2_Resistor:1608_220R
Changed lines of the file:
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@@
 	(title_block
 		(title "V2 dmx")
-		(date "2026-04-14")
+		(date "2026-05-11")
 		(rev "2026-03-30")
 		(company "Versio Duo")
