File: hardware/dmx.kicad_pcb (KiCad board)
At the start: 4 copper layers, 70 x 70 mm, 63 parts, among them J101 Cortex, J102 DX07S016JA3, J201 SJ2-25404B-SMT-TR, J301 SJ2-25404B-SMT-TR, SW101 SKSG, SW102 SKSG, U101 TPS78433QWDRBRQ1, U102 ATSAMD51G, U201 THVD2442, U301 TLP2361, Y101 32k768

Commit message: Update
Other:
- board text removed: "2026-02-07 stencil"
Changed lines of the file:
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@@
 		(layer "Edge.Cuts")
-	)
-	(gr_text "2026-02-07 stencil\n"
-		(at 117 40 0)
-		(layer "F.Fab")
-		(effects
-			(font
-				(size 0.5 0.5)
-				(thickness 0.0625)
-			)
-			(justify left bottom)
-		)
 	)
 	(segment

Commit message: Replace diode
Parts:
- D301: value RB501SM -> PMEG2010EPK; footprint V2_Diode_SMD:D_SOD-523 -> V2_Diode_SMD:D_SOD-1608
Connections:
- net Shield renamed /Shield

Commit message: Update
Parts:
- renumbered C108 to C101, C109 to C102, C101 to C103, C102 to C104, C103 to C105, C104 to C106, C105 to C107, C106 to C108, C107 to C109, C302 to C301, C301 to C302, D103 to D101, D101 to D102, D102 to D103, D405 to D402, D409 to D403, D413 to D404, D402 to D405, D410 to D407, D414 to D408, D403 to D409, D407 to D410, D415 to D412, D404 to D413, D408 to D414, D412 to D415, ICON104 to ICON101, ICON101 to ICON103, ICON103 to ICON104, INFO102 to INFO101, INFO101 to INFO102, R104 to R101, R101 to R102, R102 to R103, R103 to R104, SW102 to SW101, SW101 to SW102, U102 to U101, U101 to U102

Commit message: Good Bye Imperial
Parts:
- C101, C102, C103, C104, C105, C106, C107, C201, C301, C302: footprint V2_Capacitor_SMD:C_0603 -> V2_Capacitor_SMD:C_1608
- C108, C109: footprint V2_Capacitor_SMD:C_0805 -> V2_Capacitor_SMD:C_2012
- D101: footprint V2_LED:LED_0603 -> V2_LED:LED_1608
- R101, R102, R103, R104, R301: footprint V2_Resistor_SMD:R_0603 -> V2_Resistor_SMD:R_1608
