File: hardware/dmx.kicad_sch (KiCad schematic)
At the start: 38 parts, among them J101 Cortex, J102 DX07S016JA3, SW101 SKSG, SW102 SKSG, U101 ATSAMD51G, U102 TPS78433QWDRBRQ1, Y101 32k768

Commit message: Refresh
Parts:
- INFO102: value Layer_Numbers -> Layer_Numbers-4; footprint V2_Production:Layer_Numbers -> V2_Production:Layer_Numbers-4; symbol V2_Production:Layer_Numbers -> V2_Production:Layer_Numbers-4
Other:
- moved on the sheet: ICON101, ICON102
Changed lines of the file:
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@@
 	(title_block
 		(title "V2 dmx")
-		(date "2026-05-19")
+		(date "2026-05-27")
 		(rev "2026-03-30")
 		(company "Versio Duo")
@@
 		(unit 1)
 		(body_style 1)
-		(exclude_from_sim no)
+		(exclude_from_sim yes)
 		(in_bom no)
 		(on_board yes)
@@
 			)
 		)
-		(property "Sim.Enable" "0"
-			(at 250.19 154.94 0)
-			(hide yes)
-			(show_name no)
-			(do_not_autoplace no)
-			(effects
-				(font
-					(size 1.27 1.27)
-				)
-			)
-		)
 		(instances
 			(project "dmx"
@@
 				(font
 					(size 1.27 1.27)
+					(color 255 92 187 1)
 				)
 			)
@@
 		)
 		(property "Value" "Shield"
-			(at 262.382 86.106 90)
+			(at 263.652 86.36 90)
 			(show_name no)
 			(do_not_autoplace no)
@@
 		(in_pos_files yes)
 		(dnp no)
-		(fields_autoplaced yes)
 		(property "Reference" "#PWR0128"
 			(at 259.08 105.41 0)
@@
 		)
 		(property "Value" "+5V"
-			(at 266.7 105.4099 90)
+			(at 268.732 105.4099 90)
 			(show_name no)
 			(do_not_autoplace no)
@@
 				(font
 					(size 1.27 1.27)
+					(color 255 92 187 1)
 				)
-				(justify left)
 			)
 		)
@@
 		(unit 1)
 		(body_style 1)
-		(exclude_from_sim no)
+		(exclude_from_sim yes)
 		(in_bom no)
 		(on_board yes)
@@
 			)
 		)
-		(property "Sim.Enable" "0"
-			(at 200.66 162.56 0)
-			(hide yes)
-			(show_name no)
-			(do_not_autoplace no)
-			(effects
-				(font
-					(size 1.27 1.27)
-				)
-			)
-		)
 		(instances
 			(project "dmx"
@@
 		)
 		(property "Value" "+3V3"
-			(at 75.946 16.764 0)
+			(at 78.74 16.256 0)
 			(show_name no)
 			(do_not_autoplace no)
@@
 				(font
 					(size 1.27 1.27)
+					(color 255 92 187 1)
 				)
-				(justify left)
 			)
 		)
@@
 				(font
 					(size 1.27 1.27)
+					(color 255 92 187 1)
 				)
 			)
@@
 				(font
 					(size 1.27 1.27)
+					(color 255 92 187 1)
 				)
 			)
@@
 				(font
 					(size 1.27 1.27)
+					(color 255 92 187 1)
 				)
 			)
@@
 				(font
 					(size 1.27 1.27)
+					(color 255 92 187 1)
 				)
 			)
@@
 		(in_pos_files yes)
 		(dnp no)
-		(fields_autoplaced yes)
 		(property "Reference" "#PWR0110"
 			(at 120.65 92.71 0)
@@
 		)
 		(property "Value" "+3V3"
-			(at 115.57 90.17 90)
+			(at 110.236 92.71 90)
 			(show_name no)
 			(do_not_autoplace no)
@@
 				(font
 					(size 1.27 1.27)
+					(color 255 92 187 1)
 				)
 			)
@@
 	)
 	(symbol
-		(lib_id "V2_Production:Layer_Numbers")
+		(lib_id "V2_Production:Layer_Numbers-4")
 		(at 201.93 176.53 0)
 		(unit 1)
@@
 			)
 		)
-		(property "Value" "Layer_Numbers"
+		(property "Value" "Layer_Numbers-4"
 			(at 203.8684 173.0585 0)
 			(hide yes)
@@
 			)
 		)
-		(property "Footprint" "V2_Production:Layer_Numbers"
+		(property "Footprint" "V2_Production:Layer_Numbers-4"
 			(at 201.93 182.88 0)
 			(hide yes)
@@
 		(in_pos_files yes)
 		(dnp no)
-		(fields_autoplaced yes)
 		(property "Reference" "#PWR0119"
 			(at 201.93 90.17 0)
@@
 		)
 		(property "Value" "+5V"
-			(at 204.47 85.0899 0)
+			(at 201.93 81.7879 0)
 			(show_name no)
 			(do_not_autoplace no)
@@
 				(font
 					(size 1.27 1.27)
+					(color 255 92 187 1)
 				)
-				(justify left)
 			)
 		)
@@
 	(symbol
 		(lib_id "V2_Artwork:Board_dmx")
-		(at 180.34 177.8 0)
+		(at 180.34 176.53 0)
 		(unit 1)
 		(body_style 1)
-		(exclude_from_sim no)
+		(exclude_from_sim yes)
 		(in_bom no)
 		(on_board yes)
@@
 		(dnp no)
 		(property "Reference" "ICON101"
-			(at 176.276 173.482 0)
+			(at 176.276 172.212 0)
 			(show_name no)
 			(do_not_autoplace no)
@@
 		)
 		(property "Value" "Board_dmx"
-			(at 177.292 173.736 0)
+			(at 177.292 172.466 0)
 			(hide yes)
 			(show_name no)
@@
 		)
 		(property "Footprint" "V2_Artwork:Board_dmx_Small"
-			(at 180.34 182.88 0)
+			(at 180.34 181.61 0)
 			(hide yes)
 			(show_name no)
@@
 		)
 		(property "Datasheet" ""
-			(at 180.34 177.8 0)
+			(at 180.34 176.53 0)
 			(hide yes)
 			(show_name no)
@@
 		)
 		(property "Description" ""
-			(at 180.34 177.8 0)
-			(hide yes)
-			(show_name no)
-			(do_not_autoplace no)
-			(effects
-				(font
-					(size 1.27 1.27)
-				)
-			)
-		)
-		(property "Sim.Enable" "0"
-			(at 180.34 177.8 0)
+			(at 180.34 176.53 0)
 			(hide yes)
 			(show_name no)
@@
 		(in_pos_files yes)
 		(dnp no)
-		(fields_autoplaced yes)
 		(property "Reference" "#PWR0125"
 			(at 251.46 78.74 0)
@@
 		)
 		(property "Value" "+5V"
-			(at 259.08 78.7399 90)
+			(at 261.112 78.7399 90)
 			(show_name no)
 			(do_not_autoplace no)
@@
 				(font
 					(size 1.27 1.27)
+					(color 255 92 187 1)
 				)
-				(justify left)
 			)
 		)
@@
 		(unit 1)
 		(body_style 1)
-		(exclude_from_sim no)
+		(exclude_from_sim yes)
 		(in_bom no)
 		(on_board yes)
@@
 			)
 		)
-		(property "Sim.Enable" "0"
-			(at 250.19 161.29 0)
-			(hide yes)
-			(show_name no)
-			(do_not_autoplace no)
-			(effects
-				(font
-					(size 1.27 1.27)
-				)
-			)
-		)
 		(instances
 			(project "dmx"
@@
 	(symbol
 		(lib_id "V2_Artwork:V2-logo")
-		(at 181.61 160.02 0)
+		(at 181.61 161.29 0)
 		(unit 1)
 		(body_style 1)
@@
 		(dnp no)
 		(property "Reference" "ICON102"
-			(at 177.8 153.67 0)
+			(at 177.8 154.94 0)
 			(show_name no)
 			(do_not_autoplace no)
@@
 		)
 		(property "Value" "V2-logo"
-			(at 177.8 156.21 0)
+			(at 177.8 157.48 0)
 			(hide yes)
 			(show_name no)
@@
 		)
 		(property "Footprint" "V2_Artwork:Logo_Small"
-			(at 181.61 167.64 0)
+			(at 181.61 168.91 0)
 			(hide yes)
 			(show_name no)
@@
 		)
 		(property "Datasheet" ""
-			(at 181.61 160.02 0)
+			(at 181.61 161.29 0)
 			(hide yes)
 			(show_name no)
@@
 		)
 		(property "Description" ""
-			(at 181.61 160.02 0)
+			(at 181.61 161.29 0)
 			(hide yes)
 			(show_name no)
